Commit message: minor changes

File: summit_xl_description/robots/summit_xl_csl.urdf.xacro (robot description, xacro)
@@ -54,5 +54,5 @@
                   <origin rpy="0.0 0.0 0.0" xyz="0 0 0.0"/>
                   <geometry>
-                    <mesh filename="package://summit_description/meshes/aluminium_channel/model.stl" scale="0.02 0.02 0.02"/>
+                    <mesh filename="package://summit_xl_description/meshes/aluminium_channel/model.stl" scale="0.02 0.02 0.02"/>
                   </geometry>
                   <material name="">
@@ -63,5 +63,5 @@
                   <origin rpy="0.0 0 0.0" xyz="0 0 0"/>
                   <geometry>
-                    <mesh filename="package://summit_description/meshes/aluminium_channel/model.stl" scale="0.02 0.02 0.02"/>
+                    <mesh filename="package://summit_xl_description/meshes/aluminium_channel/model.stl" scale="0.02 0.02 0.02"/>
                   </geometry>
                 </collision>
@@ -82,5 +82,5 @@
                   <origin rpy="0.0 0.0 0.0" xyz="0 0 0.0"/>
                   <geometry>
-                    <mesh filename="package://summit_description/meshes/aluminium_channel/model.stl" scale="0.02 0.02 0.02"/>
+                    <mesh filename="package://summit_xl_description/meshes/aluminium_channel/model.stl" scale="0.02 0.02 0.02"/>
                   </geometry>
                   <material name="">
@@ -91,5 +91,5 @@
                   <origin rpy="0.0 0 0.0" xyz="0 0 0"/>
                   <geometry>
-                    <mesh filename="package://summit_description/meshes/aluminium_channel/model.stl" scale="0.02 0.02 0.02"/>
+                    <mesh filename="package://summit_xl_description/meshes/aluminium_channel/model.stl" scale="0.02 0.02 0.02"/>
                   </geometry>
                 </collision>

File: summit_xl_description/urdf/wheels/omni_wheel.urdf.xacro (robot description, xacro)
@@ -72,5 +72,5 @@
       <type>transmission_interface/SimpleTransmission</type>
       <joint name="${prefix}_wheel_joint" >
-        <hardwareInterface>VelocityJointInterface</hardwareInterface>
+        <hardwareInterface>hardware_interface/VelocityJointInterface</hardwareInterface>
       </joint>
       <actuator name="${prefix}_wheel_joint_motor">
